Commit message: 1. urdf_extended 2. publishing target pose to tf

File: urdf/moveo_ps3_extended.urdf (robot description, URDF)
Before this commit: robot moveo, 7 links, 6 joints
Links:
- added link world
Joints:
- added joint world: type fixed, parent world, child base_link, origin xyz=0 0 0.129, axis 0 0 1

Commit message: using tf for calculating target pose

File: urdf/moveo_ps3_extended.urdf (robot description, URDF)
Before this commit: robot moveo, 8 links, 7 joints
Joints:
- joint world: origin xyz=0 0 0.129 -> xyz=0 -0.22 0.040

Commit message: delete axis for fixed joints

File: urdf/moveo_ps3_extended.urdf (robot description, URDF)
Before this commit: robot moveo, 8 links, 7 joints
Joints:
- joint end_point: axis 1 0 0 -> (none)
- joint world: axis 0 0 1 -> (none)
